Commit message: Add MH5 Short & Long Variants

File: motoman_mh5_support/urdf/mh5.xacro (robot description, xacro)
@@ -1,5 +1,5 @@
 <?xml version="1.0" ?>
 <robot name="motoman_mh5" xmlns:xacro="http://ros.org/wiki/xacro">
-	<xacro:include filename="$(find motoman_mh5_support)/urdf/mh5_macro.xacro" />
-	<xacro:motoman_mh5 prefix=""/>
+  <xacro:include filename="$(find motoman_mh5_support)/urdf/mh5_macro.xacro" />
+  <xacro:motoman_mh5 prefix=""/>
 </robot>

File: motoman_mh5_support/urdf/mh5l_macro.xacro (robot description, xacro)
@@ -1,5 +1,5 @@
 <?xml version="1.0" ?>
 <robot xmlns:xacro="http://ros.org/wiki/xacro">
-  <xacro:macro name="motoman_mh5" params="prefix">
+  <xacro:macro name="motoman_mh5l" params="prefix">
     <!-- Properties -->
     <material name="yaskawa_white">
@@ -11,5 +11,5 @@
         <origin xyz="0 0 0" rpy="0 0 0" />
         <geometry>
-          <mesh filename="package://motoman_mh5_support/meshes/mh5/visual/base_link.stl" />
+          <mesh filename="package://motoman_mh5_support/meshes/mh5l/visual/base_link.stl" />
         </geometry>
         <material name="yaskawa_white"/>
@@ -18,5 +18,5 @@
         <origin xyz="0 0 0" rpy="0 0 0" />
         <geometry>
-          <mesh filename="package://motoman_mh5_support/meshes/mh5/collision/base_link.stl" />
+          <mesh filename="package://motoman_mh5_support/meshes/mh5l/collision/base_link.stl" />
         </geometry>
       </collision>
@@ -26,5 +26,5 @@
         <origin xyz="0 0 0" rpy="0 0 0" />
         <geometry>
-          <mesh filename="package://motoman_mh5_support/meshes/mh5/visual/link_1_s.stl"/>
+          <mesh filename="package://motoman_mh5_support/meshes/mh5l/visual/link_1_s.stl"/>
         </geometry>
         <material name="yaskawa_white"/>
@@ -33,5 +33,5 @@
         <origin xyz="0 0 0" rpy="0 0 0" />
         <geometry>
-          <mesh filename="package://motoman_mh5_support/meshes/mh5/collision/link_1_s.stl" />
+          <mesh filename="package://motoman_mh5_support/meshes/mh5l/collision/link_1_s.stl" />
         </geometry>
       </collision>
@@ -41,5 +41,5 @@
         <origin xyz="0 0 0" rpy="0 0 0" />
         <geometry>
-          <mesh filename="package://motoman_mh5_support/meshes/mh5/visual/link_2_l.stl"/>
+          <mesh filename="package://motoman_mh5_support/meshes/mh5l/visual/link_2_l.stl"/>
         </geometry>
         <material name="yaskawa_white"/>
@@ -48,5 +48,5 @@
         <origin xyz="0 0 0" rpy="0 0 0" />
         <geometry>
-          <mesh filename="package://motoman_mh5_support/meshes/mh5/collision/link_2_l.stl" />
+          <mesh filename="package://motoman_mh5_support/meshes/mh5l/collision/link_2_l.stl" />
         </geometry>
       </collision>
@@ -56,5 +56,5 @@
         <origin xyz="0 0 0" rpy="0 0 0" />
         <geometry>
-          <mesh filename="package://motoman_mh5_support/meshes/mh5/visual/link_3_u.stl"/>
+          <mesh filename="package://motoman_mh5_support/meshes/mh5l/visual/link_3_u.stl"/>
         </geometry>
         <material name="yaskawa_white"/>
@@ -63,5 +63,5 @@
         <origin xyz="0 0 0" rpy="0 0 0" />
         <geometry>
-          <mesh filename="package://motoman_mh5_support/meshes/mh5/collision/link_3_u.stl" />
+          <mesh filename="package://motoman_mh5_support/meshes/mh5l/collision/link_3_u.stl" />
         </geometry>
       </collision>
@@ -71,5 +71,5 @@
         <origin xyz="0 0 0" rpy="0 0 0" />
         <geometry>
-          <mesh filename="package://motoman_mh5_support/meshes/mh5/visual/link_4_r.stl"/>
+          <mesh filename="package://motoman_mh5_support/meshes/mh5l/visual/link_4_r.stl"/>
         </geometry>
         <material name="yaskawa_white"/>
@@ -78,5 +78,5 @@
         <origin xyz="0 0 0" rpy="0 0 0" />
         <geometry>
-          <mesh filename="package://motoman_mh5_support/meshes/mh5/collision/link_4_r.stl" />
+          <mesh filename="package://motoman_mh5_support/meshes/mh5l/collision/link_4_r.stl" />
         </geometry>
       </collision>
@@ -86,5 +86,5 @@
         <origin xyz="0 0 0" rpy="0 0 0" />
         <geometry>
-          <mesh filename="package://motoman_mh5_support/meshes/mh5/visual/link_5_b.stl"/>
+          <mesh filename="package://motoman_mh5_support/meshes/mh5l/visual/link_5_b.stl"/>
         </geometry>
         <material name="yaskawa_white"/>
@@ -93,5 +93,5 @@
         <origin xyz="0 0 0" rpy="0 0 0" />
         <geometry>
-          <mesh filename="package://motoman_mh5_support/meshes/mh5/collision/link_5_b.stl" />
+          <mesh filename="package://motoman_mh5_support/meshes/mh5l/collision/link_5_b.stl" />
         </geometry>
       </collision>
@@ -101,5 +101,5 @@
         <origin xyz="0 0 0" rpy="0 0 0" />
         <geometry>
-          <mesh filename="package://motoman_mh5_support/meshes/mh5/visual/link_6_t.stl" />
+          <mesh filename="package://motoman_mh5_support/meshes/mh5l/visual/link_6_t.stl" />
         </geometry>
         <material name="yaskawa_white"/>
@@ -108,5 +108,5 @@
         <origin xyz="0 0 0" rpy="0 0 0" />
         <geometry>
-          <mesh filename="package://motoman_mh5_support/meshes/mh5/collision/link_6_t.stl" />
+          <mesh filename="package://motoman_mh5_support/meshes/mh5l/collision/link_6_t.stl" />
         </geometry>
       </collision>
@@ -119,5 +119,5 @@
       <origin xyz="0 0 0.330" rpy="0 0 0"/>
       <axis xyz="0 0 1" />
-      <limit lower="-${radians(170)}" upper="${radians(170)}" effort="215.6" velocity="${radians(376)}" />
+      <limit lower="-${radians(170)}" upper="${radians(170)}" effort="303.8" velocity="${radians(270)}" />
     </joint>
     <joint name="${prefix}joint_2_l" type="revolute">
@@ -126,12 +126,12 @@
       <origin xyz="0.0880 0 0.00" rpy="0 0 0"/>
       <axis xyz="0 1 0" />
-      <limit lower="-${radians(65)}" upper="${radians(150)}" effort="176.4" velocity="${radians(350)}" />
+      <limit lower="-${radians(65)}" upper="${radians(150)}" effort="205.8" velocity="${radians(280)}" />
     </joint>
     <joint name="${prefix}joint_3_u" type="revolute">
       <parent link="${prefix}link_2_l"/>
       <child link="${prefix}link_3_u"/>
-      <origin xyz="0 0 0.310" rpy="0 0 0"/>
+      <origin xyz="0 0 0.400" rpy="0 0 0"/>
       <axis xyz="0 -1 0" />
-      <limit lower="-${radians(70)}" upper="${radians(190)}" effort="76.8" velocity="${radians(400)}" />
+      <limit lower="-${radians(70)}" upper="${radians(190)}" effort="85.5" velocity="${radians(300)}" />
     </joint>
     <joint name="${prefix}joint_4_r" type="revolute">
@@ -145,5 +145,5 @@
       <parent link="${prefix}link_4_r"/>
       <child link="${prefix}link_5_b"/>
-      <origin xyz="0.305 0 0" rpy="0 0 0"/>
+      <origin xyz="0.405 0 0" rpy="0 0 0"/>
       <axis xyz="0 -1 0" />
       <limit lower="-${radians(135)}" upper="${radians(135)}" effort="18.0" velocity="${radians(450)}" />
@@ -152,5 +152,5 @@
       <parent link="${prefix}link_5_b"/>
       <child link="${prefix}link_6_t"/>
-      <origin xyz="0.0865 0 0" rpy="0 0 0"/>
+      <origin xyz="0.080 0 0" rpy="0 0 0"/>
       <axis xyz="-1 0 0" />
       <limit lower="-${radians(360)}" upper="${radians(360)}" effort="18.0" velocity="${radians(720)}" />
