Commit message: Removed Duplicate Meshes
Link meshes for the MH5L matching those of the MH5 were removed.
Effected URDF references redirected to MH5 meshes.
Moved unique "link-s" mesh to dedicated mh5_old_variants directory.
Updated changelog to reflect shared meshes.

File: motoman_mh5_support/urdf/mh5_macro.xacro (robot description, xacro)
@@ -57,4 +57,5 @@
         <geometry>
           <mesh filename="package://motoman_mh5_support/meshes/mh5/visual/link_3_u.stl"/>
+          <!-- <mesh filename="package://motoman_mh5_support/meshes/mh5_old_variants/visual/link_3_u.stl"/> --><!-- Uncomment & switch with above to use alternative U-link. -->
         </geometry>
         <material name="yaskawa_white"/>
@@ -64,4 +65,5 @@
         <geometry>
           <mesh filename="package://motoman_mh5_support/meshes/mh5/collision/link_3_u.stl" />
+          <!-- <mesh filename="package://motoman_mh5_support/meshes/mh5_old_variants/collision/link_3_u.stl" /> --><!-- Uncomment & switch with above to use alternative U-link. -->
         </geometry>
       </collision>

File: motoman_mh5_support/urdf/mh5l_macro.xacro (robot description, xacro)
@@ -11,5 +11,5 @@
         <origin xyz="0 0 0" rpy="0 0 0" />
         <geometry>
-          <mesh filename="package://motoman_mh5_support/meshes/mh5l/visual/base_link.stl" />
+          <mesh filename="package://motoman_mh5_support/meshes/mh5/visual/base_link.stl" />
         </geometry>
         <material name="yaskawa_white"/>
@@ -18,5 +18,5 @@
         <origin xyz="0 0 0" rpy="0 0 0" />
         <geometry>
-          <mesh filename="package://motoman_mh5_support/meshes/mh5l/collision/base_link.stl" />
+          <mesh filename="package://motoman_mh5_support/meshes/mh5/collision/base_link.stl" />
         </geometry>
       </collision>
@@ -26,5 +26,5 @@
         <origin xyz="0 0 0" rpy="0 0 0" />
         <geometry>
-          <mesh filename="package://motoman_mh5_support/meshes/mh5l/visual/link_1_s.stl"/>
+          <mesh filename="package://motoman_mh5_support/meshes/mh5/visual/link_1_s.stl"/>
         </geometry>
         <material name="yaskawa_white"/>
@@ -33,5 +33,5 @@
         <origin xyz="0 0 0" rpy="0 0 0" />
         <geometry>
-          <mesh filename="package://motoman_mh5_support/meshes/mh5l/collision/link_1_s.stl" />
+          <mesh filename="package://motoman_mh5_support/meshes/mh5/collision/link_1_s.stl" />
         </geometry>
       </collision>
@@ -56,5 +56,5 @@
         <origin xyz="0 0 0" rpy="0 0 0" />
         <geometry>
-          <mesh filename="package://motoman_mh5_support/meshes/mh5l/visual/link_3_u.stl"/>
+          <mesh filename="package://motoman_mh5_support/meshes/mh5/visual/link_3_u.stl"/>
         </geometry>
         <material name="yaskawa_white"/>
@@ -63,5 +63,5 @@
         <origin xyz="0 0 0" rpy="0 0 0" />
         <geometry>
-          <mesh filename="package://motoman_mh5_support/meshes/mh5l/collision/link_3_u.stl" />
+          <mesh filename="package://motoman_mh5_support/meshes/mh5/collision/link_3_u.stl" />
         </geometry>
       </collision>
@@ -86,5 +86,5 @@
         <origin xyz="0 0 0" rpy="0 0 0" />
         <geometry>
-          <mesh filename="package://motoman_mh5_support/meshes/mh5l/visual/link_5_b.stl"/>
+          <mesh filename="package://motoman_mh5_support/meshes/mh5/visual/link_5_b.stl"/>
         </geometry>
         <material name="yaskawa_white"/>
@@ -93,5 +93,5 @@
         <origin xyz="0 0 0" rpy="0 0 0" />
         <geometry>
-          <mesh filename="package://motoman_mh5_support/meshes/mh5l/collision/link_5_b.stl" />
+          <mesh filename="package://motoman_mh5_support/meshes/mh5/collision/link_5_b.stl" />
         </geometry>
       </collision>
@@ -101,5 +101,5 @@
         <origin xyz="0 0 0" rpy="0 0 0" />
         <geometry>
-          <mesh filename="package://motoman_mh5_support/meshes/mh5l/visual/link_6_t.stl" />
+          <mesh filename="package://motoman_mh5_support/meshes/mh5/visual/link_6_t.stl" />
         </geometry>
         <material name="yaskawa_white"/>
@@ -108,5 +108,5 @@
         <origin xyz="0 0 0" rpy="0 0 0" />
         <geometry>
-          <mesh filename="package://motoman_mh5_support/meshes/mh5l/collision/link_6_t.stl" />
+          <mesh filename="package://motoman_mh5_support/meshes/mh5/collision/link_6_t.stl" />
         </geometry>
       </collision>

Commit message: mh5/mh5l: use materials from resources package

File: motoman_mh5_support/urdf/mh5_macro.xacro (robot description, xacro)
@@ -2,8 +2,5 @@
 <robot xmlns:xacro="http://ros.org/wiki/xacro">
   <xacro:macro name="motoman_mh5" params="prefix">
-    <!-- Properties -->
-    <material name="yaskawa_white">
-      <color rgba="0.9 0.9 0.9 1" />
-    </material>
+    <xacro:include filename="$(find motoman_resources)/urdf/common_materials.xacro"/>
     <!-- link list -->
     <link name="${prefix}base_link">
@@ -13,5 +10,5 @@
           <mesh filename="package://motoman_mh5_support/meshes/mh5/visual/base_link.stl" />
         </geometry>
-        <material name="yaskawa_white"/>
+        <xacro:material_yaskawa_white/>
       </visual>
       <collision>
@@ -28,5 +25,5 @@
           <mesh filename="package://motoman_mh5_support/meshes/mh5/visual/link_1_s.stl"/>
         </geometry>
-        <material name="yaskawa_white"/>
+        <xacro:material_yaskawa_white/>
       </visual>
       <collision>
@@ -43,5 +40,5 @@
           <mesh filename="package://motoman_mh5_support/meshes/mh5/visual/link_2_l.stl"/>
         </geometry>
-        <material name="yaskawa_white"/>
+        <xacro:material_yaskawa_white/>
       </visual>
       <collision>
@@ -59,5 +56,5 @@
           <!-- <mesh filename="package://motoman_mh5_support/meshes/mh5_old_variants/visual/link_3_u.stl"/> --><!-- Uncomment & switch with above to use alternative U-link. -->
         </geometry>
-        <material name="yaskawa_white"/>
+        <xacro:material_yaskawa_white/>
       </visual>
       <collision>
@@ -75,5 +72,5 @@
           <mesh filename="package://motoman_mh5_support/meshes/mh5/visual/link_4_r.stl"/>
         </geometry>
-        <material name="yaskawa_white"/>
+        <xacro:material_yaskawa_white/>
       </visual>
       <collision>
@@ -90,5 +87,5 @@
           <mesh filename="package://motoman_mh5_support/meshes/mh5/visual/link_5_b.stl"/>
         </geometry>
-        <material name="yaskawa_white"/>
+        <xacro:material_yaskawa_white/>
       </visual>
       <collision>
@@ -105,5 +102,5 @@
           <mesh filename="package://motoman_mh5_support/meshes/mh5/visual/link_6_t.stl" />
         </geometry>
-        <material name="yaskawa_white"/>
+        <xacro:material_yaskawa_white/>
       </visual>
       <collision>

File: motoman_mh5_support/urdf/mh5l_macro.xacro (robot description, xacro)
@@ -2,8 +2,5 @@
 <robot xmlns:xacro="http://ros.org/wiki/xacro">
   <xacro:macro name="motoman_mh5l" params="prefix">
-    <!-- Properties -->
-    <material name="yaskawa_white">
-      <color rgba="0.9 0.9 0.9 1" />
-    </material>
+    <xacro:include filename="$(find motoman_resources)/urdf/common_materials.xacro"/>
     <!-- link list -->
     <link name="${prefix}base_link">
@@ -13,5 +10,5 @@
           <mesh filename="package://motoman_mh5_support/meshes/mh5/visual/base_link.stl" />
         </geometry>
-        <material name="yaskawa_white"/>
+        <xacro:material_yaskawa_white/>
       </visual>
       <collision>
@@ -28,5 +25,5 @@
           <mesh filename="package://motoman_mh5_support/meshes/mh5/visual/link_1_s.stl"/>
         </geometry>
-        <material name="yaskawa_white"/>
+        <xacro:material_yaskawa_white/>
       </visual>
       <collision>
@@ -43,5 +40,5 @@
           <mesh filename="package://motoman_mh5_support/meshes/mh5l/visual/link_2_l.stl"/>
         </geometry>
-        <material name="yaskawa_white"/>
+        <xacro:material_yaskawa_white/>
       </visual>
       <collision>
@@ -58,5 +55,5 @@
           <mesh filename="package://motoman_mh5_support/meshes/mh5/visual/link_3_u.stl"/>
         </geometry>
-        <material name="yaskawa_white"/>
+        <xacro:material_yaskawa_white/>
       </visual>
       <collision>
@@ -73,5 +70,5 @@
           <mesh filename="package://motoman_mh5_support/meshes/mh5l/visual/link_4_r.stl"/>
         </geometry>
-        <material name="yaskawa_white"/>
+        <xacro:material_yaskawa_white/>
       </visual>
       <collision>
@@ -88,5 +85,5 @@
           <mesh filename="package://motoman_mh5_support/meshes/mh5/visual/link_5_b.stl"/>
         </geometry>
-        <material name="yaskawa_white"/>
+        <xacro:material_yaskawa_white/>
       </visual>
       <collision>
@@ -103,5 +100,5 @@
           <mesh filename="package://motoman_mh5_support/meshes/mh5/visual/link_6_t.stl" />
         </geometry>
-        <material name="yaskawa_white"/>
+        <xacro:material_yaskawa_white/>
       </visual>
       <collision>

Commit message: fix MH5 joint6 offset: 80mm per datasheet and spec
see table at https://github.com/ros-industrial/motoman/issues/377#issuecomment-742556746

File: motoman_mh5_support/urdf/mh5_macro.xacro (robot description, xacro)
@@ -151,5 +151,5 @@
       <parent link="${prefix}link_5_b"/>
       <child link="${prefix}link_6_t"/>
-      <origin xyz="0.0865 0 0" rpy="0 0 0"/>
+      <origin xyz="0.080 0 0" rpy="0 0 0"/>
       <axis xyz="-1 0 0" />
       <limit lower="-${radians(360)}" upper="${radians(360)}" effort="18.0" velocity="${radians(720)}" />
