Commit message: GP4 corrections and collision model update
GP4 corrections and collision model update

File: motoman_gp4_support/urdf/gp4_macro.xacro (robot description, xacro)
@@ -7,5 +7,5 @@
       <visual>
         <geometry>
-          <mesh filename="package://motoman_gp4_support/meshes/gp4/visual/base_link.stl"/>
+          <mesh filename="package://motoman_gp4_support/meshes/gp4/visual/base_link.dae"/>
         </geometry>
         <xacro:material_yaskawa_white/>
@@ -13,5 +13,5 @@
       <collision>
         <geometry>
-          <mesh filename="package://motoman_gp4_support/meshes/gp4/collision/base_link.stl"/>
+          <mesh filename="package://motoman_gp4_support/meshes/gp4/collision/base_link.dae"/>
         </geometry>
       </collision>
@@ -20,5 +20,5 @@
       <visual>
         <geometry>
-          <mesh filename="package://motoman_gp4_support/meshes/gp4/visual/link_1_s.stl"/>
+          <mesh filename="package://motoman_gp4_support/meshes/gp4/visual/link_1_s.dae"/>
         </geometry>
         <xacro:material_yaskawa_white/>
@@ -26,5 +26,5 @@
       <collision>
         <geometry>
-          <mesh filename="package://motoman_gp4_support/meshes/gp4/collision/link_1_s.stl"/>
+          <mesh filename="package://motoman_gp4_support/meshes/gp4/collision/link_1_s.dae"/>
         </geometry>
       </collision>
@@ -33,5 +33,5 @@
       <visual>
         <geometry>
-          <mesh filename="package://motoman_gp4_support/meshes/gp4/visual/link_2_l.stl"/>
+          <mesh filename="package://motoman_gp4_support/meshes/gp4/visual/link_2_l.dae"/>
         </geometry>
         <xacro:material_yaskawa_white/>
@@ -39,5 +39,5 @@
       <collision>
         <geometry>
-          <mesh filename="package://motoman_gp4_support/meshes/gp4/collision/link_2_l.stl"/>
+          <mesh filename="package://motoman_gp4_support/meshes/gp4/collision/link_2_l.dae"/>
         </geometry>
       </collision>
@@ -46,5 +46,5 @@
       <visual>
         <geometry>
-          <mesh filename="package://motoman_gp4_support/meshes/gp4/visual/link_3_u.stl"/>
+          <mesh filename="package://motoman_gp4_support/meshes/gp4/visual/link_3_u.dae"/>
         </geometry>
         <xacro:material_yaskawa_white/>
@@ -52,5 +52,5 @@
       <collision>
         <geometry>
-          <mesh filename="package://motoman_gp4_support/meshes/gp4/collision/link_3_u.stl"/>
+          <mesh filename="package://motoman_gp4_support/meshes/gp4/collision/link_3_u.dae"/>
         </geometry>
       </collision>
@@ -59,5 +59,5 @@
       <visual>
         <geometry>
-          <mesh filename="package://motoman_gp4_support/meshes/gp4/visual/link_4_r.stl"/>
+          <mesh filename="package://motoman_gp4_support/meshes/gp4/visual/link_4_r.dae"/>
         </geometry>
         <xacro:material_yaskawa_white/>
@@ -65,5 +65,5 @@
       <collision>
         <geometry>
-          <mesh filename="package://motoman_gp4_support/meshes/gp4/collision/link_4_r.stl"/>
+          <mesh filename="package://motoman_gp4_support/meshes/gp4/collision/link_4_r.dae"/>
         </geometry>
       </collision>
@@ -72,5 +72,5 @@
       <visual>
         <geometry>
-          <mesh filename="package://motoman_gp4_support/meshes/gp4/visual/link_5_b.stl"/>
+          <mesh filename="package://motoman_gp4_support/meshes/gp4/visual/link_5_b.dae"/>
         </geometry>
         <xacro:material_yaskawa_white/>
@@ -78,5 +78,5 @@
       <collision>
         <geometry>
-          <mesh filename="package://motoman_gp4_support/meshes/gp4/collision/link_5_b.stl"/>
+          <mesh filename="package://motoman_gp4_support/meshes/gp4/collision/link_5_b.dae"/>
         </geometry>
       </collision>
@@ -85,5 +85,5 @@
       <visual>
         <geometry>
-          <mesh filename="package://motoman_gp4_support/meshes/gp4/visual/link_6_t.stl"/>
+          <mesh filename="package://motoman_gp4_support/meshes/gp4/visual/link_6_t.dae"/>
         </geometry>
         <xacro:material_yaskawa_white/>
@@ -91,5 +91,5 @@
       <collision>
         <geometry>
-          <mesh filename="package://motoman_gp4_support/meshes/gp4/collision/link_6_t.stl"/>
+          <mesh filename="package://motoman_gp4_support/meshes/gp4/collision/link_6_t.dae"/>
         </geometry>
       </collision>
@@ -103,5 +103,5 @@
       <origin xyz="0 0 0.330" rpy="0 0 0" />
       <axis xyz="0 0 1" />
-      <limit lower="${radians(-170)}" upper="${radians(170)}" effort="917.28" velocity="${radians(465)}"/>
+      <limit lower="${radians(-170)}" upper="${radians(170)}" effort="220.5" velocity="${radians(465)}"/>
     </joint>
     <joint name="${prefix}joint_2_l" type="revolute">
@@ -110,5 +110,5 @@
       <origin xyz="0 0 0" rpy="0 0 0" />
       <axis xyz="0 1 0" />
-      <limit lower="${radians(-110)}" upper="${radians(130)}" effort="1223.04" velocity="${radians(465)}"/>
+      <limit lower="${radians(-110)}" upper="${radians(130)}" effort="305.76" velocity="${radians(465)}"/>
     </joint>
     <joint name="${prefix}joint_3_u" type="revolute">
@@ -117,5 +117,5 @@
       <origin xyz="0 0 0.260" rpy="0 0 0" />
       <axis xyz="0 -1 0" />
-      <limit lower="${radians(-65)}" upper="${radians(200)}" effort="642.88" velocity="${radians(525)}"/>
+      <limit lower="${radians(-65)}" upper="${radians(200)}" effort="95.55" velocity="${radians(525)}"/>
     </joint>
     <joint name="${prefix}joint_4_r" type="revolute">
@@ -124,5 +124,5 @@
       <origin xyz="0.290 0 0.015" rpy="0 0 0" />
       <axis xyz="-1 0 0" />
-      <limit lower="${radians(-200)}" upper="${radians(200)}" effort="368.48" velocity="${radians(565)}"/>
+      <limit lower="${radians(-200)}" upper="${radians(200)}" effort="48.02" velocity="${radians(565)}"/>
     </joint>
     <joint name="${prefix}joint_5_b" type="revolute">
@@ -131,5 +131,5 @@
       <origin xyz="0 0 0" rpy="0 0 0" />
       <axis xyz="0 -1 0" />
-      <limit lower="${radians(-123)}" upper="${radians(123)}" effort="141.12" velocity="${radians(565)}"/>
+      <limit lower="${radians(-123)}" upper="${radians(123)}" effort="38.42" velocity="${radians(565)}"/>
     </joint>
     <joint name="${prefix}joint_6_t" type="revolute">
@@ -138,5 +138,5 @@
       <origin xyz="0 0 0" rpy="0 0 0" />
       <axis xyz="-1 0 0" />
-      <limit lower="${radians(-455)}" upper="${radians(455)}" effort="141.12" velocity="${radians(1000)}"/>
+      <limit lower="${radians(-455)}" upper="${radians(455)}" effort="16.46" velocity="${radians(1000)}"/>
     </joint>
     <joint name="${prefix}joint_6_t-tool0" type="fixed">

Commit message: Change models from dae to stl
Change models from dae to stl

File: motoman_gp4_support/urdf/gp4_macro.xacro (robot description, xacro)
@@ -7,11 +7,11 @@
       <visual>
         <geometry>
-          <mesh filename="package://motoman_gp4_support/meshes/gp4/visual/base_link.dae"/>
+          <mesh filename="package://motoman_gp4_support/meshes/gp4/visual/base_link.stl"/>
         </geometry>
-        <xacro:material_yaskawa_white/>
+        <xacro:material_yaskawa_blue/>
       </visual>
       <collision>
         <geometry>
-          <mesh filename="package://motoman_gp4_support/meshes/gp4/collision/base_link.dae"/>
+          <mesh filename="package://motoman_gp4_support/meshes/gp4/collision/base_link.stl"/>
         </geometry>
       </collision>
@@ -20,11 +20,11 @@
       <visual>
         <geometry>
-          <mesh filename="package://motoman_gp4_support/meshes/gp4/visual/link_1_s.dae"/>
+          <mesh filename="package://motoman_gp4_support/meshes/gp4/visual/link_1_s.stl"/>
         </geometry>
-        <xacro:material_yaskawa_white/>
+        <xacro:material_yaskawa_blue/>
       </visual>
       <collision>
         <geometry>
-          <mesh filename="package://motoman_gp4_support/meshes/gp4/collision/link_1_s.dae"/>
+          <mesh filename="package://motoman_gp4_support/meshes/gp4/collision/link_1_s.stl"/>
         </geometry>
       </collision>
@@ -33,11 +33,11 @@
       <visual>
         <geometry>
-          <mesh filename="package://motoman_gp4_support/meshes/gp4/visual/link_2_l.dae"/>
+          <mesh filename="package://motoman_gp4_support/meshes/gp4/visual/link_2_l.stl"/>
         </geometry>
-        <xacro:material_yaskawa_white/>
+        <xacro:material_yaskawa_blue/>
       </visual>
       <collision>
         <geometry>
-          <mesh filename="package://motoman_gp4_support/meshes/gp4/collision/link_2_l.dae"/>
+          <mesh filename="package://motoman_gp4_support/meshes/gp4/collision/link_2_l.stl"/>
         </geometry>
       </collision>
@@ -46,11 +46,11 @@
       <visual>
         <geometry>
-          <mesh filename="package://motoman_gp4_support/meshes/gp4/visual/link_3_u.dae"/>
+          <mesh filename="package://motoman_gp4_support/meshes/gp4/visual/link_3_u.stl"/>
         </geometry>
-        <xacro:material_yaskawa_white/>
+        <xacro:material_yaskawa_blue/>
       </visual>
       <collision>
         <geometry>
-          <mesh filename="package://motoman_gp4_support/meshes/gp4/collision/link_3_u.dae"/>
+          <mesh filename="package://motoman_gp4_support/meshes/gp4/collision/link_3_u.stl"/>
         </geometry>
       </collision>
@@ -59,11 +59,11 @@
       <visual>
         <geometry>
-          <mesh filename="package://motoman_gp4_support/meshes/gp4/visual/link_4_r.dae"/>
+          <mesh filename="package://motoman_gp4_support/meshes/gp4/visual/link_4_r.stl"/>
         </geometry>
-        <xacro:material_yaskawa_white/>
+        <xacro:material_yaskawa_blue/>
       </visual>
       <collision>
         <geometry>
-          <mesh filename="package://motoman_gp4_support/meshes/gp4/collision/link_4_r.dae"/>
+          <mesh filename="package://motoman_gp4_support/meshes/gp4/collision/link_4_r.stl"/>
         </geometry>
       </collision>
@@ -72,11 +72,11 @@
       <visual>
         <geometry>
-          <mesh filename="package://motoman_gp4_support/meshes/gp4/visual/link_5_b.dae"/>
+          <mesh filename="package://motoman_gp4_support/meshes/gp4/visual/link_5_b.stl"/>
         </geometry>
-        <xacro:material_yaskawa_white/>
+        <xacro:material_yaskawa_blue/>
       </visual>
       <collision>
         <geometry>
-          <mesh filename="package://motoman_gp4_support/meshes/gp4/collision/link_5_b.dae"/>
+          <mesh filename="package://motoman_gp4_support/meshes/gp4/collision/link_5_b.stl"/>
         </geometry>
       </collision>
@@ -85,11 +85,11 @@
       <visual>
         <geometry>
-          <mesh filename="package://motoman_gp4_support/meshes/gp4/visual/link_6_t.dae"/>
+          <mesh filename="package://motoman_gp4_support/meshes/gp4/visual/link_6_t.stl"/>
         </geometry>
-        <xacro:material_yaskawa_white/>
+        <xacro:material_yaskawa_silver/>
       </visual>
       <collision>
         <geometry>
-          <mesh filename="package://motoman_gp4_support/meshes/gp4/collision/link_6_t.dae"/>
+          <mesh filename="package://motoman_gp4_support/meshes/gp4/collision/link_6_t.stl"/>
         </geometry>
       </collision>

Commit message: Revert "Change models from dae to stl"
This reverts commit ec43aaddbbf2e4f09222170db85d6b9c7745cda2.

File: motoman_gp4_support/urdf/gp4_macro.xacro (robot description, xacro)
@@ -7,11 +7,11 @@
       <visual>
         <geometry>
-          <mesh filename="package://motoman_gp4_support/meshes/gp4/visual/base_link.stl"/>
+          <mesh filename="package://motoman_gp4_support/meshes/gp4/visual/base_link.dae"/>
         </geometry>
-        <xacro:material_yaskawa_blue/>
+        <xacro:material_yaskawa_white/>
       </visual>
       <collision>
         <geometry>
-          <mesh filename="package://motoman_gp4_support/meshes/gp4/collision/base_link.stl"/>
+          <mesh filename="package://motoman_gp4_support/meshes/gp4/collision/base_link.dae"/>
         </geometry>
       </collision>
@@ -20,11 +20,11 @@
       <visual>
         <geometry>
-          <mesh filename="package://motoman_gp4_support/meshes/gp4/visual/link_1_s.stl"/>
+          <mesh filename="package://motoman_gp4_support/meshes/gp4/visual/link_1_s.dae"/>
         </geometry>
-        <xacro:material_yaskawa_blue/>
+        <xacro:material_yaskawa_white/>
       </visual>
       <collision>
         <geometry>
-          <mesh filename="package://motoman_gp4_support/meshes/gp4/collision/link_1_s.stl"/>
+          <mesh filename="package://motoman_gp4_support/meshes/gp4/collision/link_1_s.dae"/>
         </geometry>
       </collision>
@@ -33,11 +33,11 @@
       <visual>
         <geometry>
-          <mesh filename="package://motoman_gp4_support/meshes/gp4/visual/link_2_l.stl"/>
+          <mesh filename="package://motoman_gp4_support/meshes/gp4/visual/link_2_l.dae"/>
         </geometry>
-        <xacro:material_yaskawa_blue/>
+        <xacro:material_yaskawa_white/>
       </visual>
       <collision>
         <geometry>
-          <mesh filename="package://motoman_gp4_support/meshes/gp4/collision/link_2_l.stl"/>
+          <mesh filename="package://motoman_gp4_support/meshes/gp4/collision/link_2_l.dae"/>
         </geometry>
       </collision>
@@ -46,11 +46,11 @@
       <visual>
         <geometry>
-          <mesh filename="package://motoman_gp4_support/meshes/gp4/visual/link_3_u.stl"/>
+          <mesh filename="package://motoman_gp4_support/meshes/gp4/visual/link_3_u.dae"/>
         </geometry>
-        <xacro:material_yaskawa_blue/>
+        <xacro:material_yaskawa_white/>
       </visual>
       <collision>
         <geometry>
-          <mesh filename="package://motoman_gp4_support/meshes/gp4/collision/link_3_u.stl"/>
+          <mesh filename="package://motoman_gp4_support/meshes/gp4/collision/link_3_u.dae"/>
         </geometry>
       </collision>
@@ -59,11 +59,11 @@
       <visual>
         <geometry>
-          <mesh filename="package://motoman_gp4_support/meshes/gp4/visual/link_4_r.stl"/>
+          <mesh filename="package://motoman_gp4_support/meshes/gp4/visual/link_4_r.dae"/>
         </geometry>
-        <xacro:material_yaskawa_blue/>
+        <xacro:material_yaskawa_white/>
       </visual>
       <collision>
         <geometry>
-          <mesh filename="package://motoman_gp4_support/meshes/gp4/collision/link_4_r.stl"/>
+          <mesh filename="package://motoman_gp4_support/meshes/gp4/collision/link_4_r.dae"/>
         </geometry>
       </collision>
@@ -72,11 +72,11 @@
       <visual>
         <geometry>
-          <mesh filename="package://motoman_gp4_support/meshes/gp4/visual/link_5_b.stl"/>
+          <mesh filename="package://motoman_gp4_support/meshes/gp4/visual/link_5_b.dae"/>
         </geometry>
-        <xacro:material_yaskawa_blue/>
+        <xacro:material_yaskawa_white/>
       </visual>
       <collision>
         <geometry>
-          <mesh filename="package://motoman_gp4_support/meshes/gp4/collision/link_5_b.stl"/>
+          <mesh filename="package://motoman_gp4_support/meshes/gp4/collision/link_5_b.dae"/>
         </geometry>
       </collision>
@@ -85,11 +85,11 @@
       <visual>
         <geometry>
-          <mesh filename="package://motoman_gp4_support/meshes/gp4/visual/link_6_t.stl"/>
+          <mesh filename="package://motoman_gp4_support/meshes/gp4/visual/link_6_t.dae"/>
         </geometry>
-        <xacro:material_yaskawa_silver/>
+        <xacro:material_yaskawa_white/>
       </visual>
       <collision>
         <geometry>
-          <mesh filename="package://motoman_gp4_support/meshes/gp4/collision/link_6_t.stl"/>
+          <mesh filename="package://motoman_gp4_support/meshes/gp4/collision/link_6_t.dae"/>
         </geometry>
       </collision>

Commit message: Change collision model to stl and left visual models as dae
Change collision model to stl and left visual models as dae

File: motoman_gp4_support/urdf/gp4_macro.xacro (robot description, xacro)
@@ -9,9 +9,9 @@
           <mesh filename="package://motoman_gp4_support/meshes/gp4/visual/base_link.dae"/>
         </geometry>
-        <xacro:material_yaskawa_white/>
+        <xacro:material_yaskawa_blue/>
       </visual>
       <collision>
         <geometry>
-          <mesh filename="package://motoman_gp4_support/meshes/gp4/collision/base_link.dae"/>
+          <mesh filename="package://motoman_gp4_support/meshes/gp4/collision/base_link.stl"/>
         </geometry>
       </collision>
@@ -22,9 +22,9 @@
           <mesh filename="package://motoman_gp4_support/meshes/gp4/visual/link_1_s.dae"/>
         </geometry>
-        <xacro:material_yaskawa_white/>
+        <xacro:material_yaskawa_blue/>
       </visual>
       <collision>
         <geometry>
-          <mesh filename="package://motoman_gp4_support/meshes/gp4/collision/link_1_s.dae"/>
+          <mesh filename="package://motoman_gp4_support/meshes/gp4/collision/link_1_s.stl"/>
         </geometry>
       </collision>
@@ -35,9 +35,9 @@
           <mesh filename="package://motoman_gp4_support/meshes/gp4/visual/link_2_l.dae"/>
         </geometry>
-        <xacro:material_yaskawa_white/>
+        <xacro:material_yaskawa_blue/>
       </visual>
       <collision>
         <geometry>
-          <mesh filename="package://motoman_gp4_support/meshes/gp4/collision/link_2_l.dae"/>
+          <mesh filename="package://motoman_gp4_support/meshes/gp4/collision/link_2_l.stl"/>
         </geometry>
       </collision>
@@ -48,9 +48,9 @@
           <mesh filename="package://motoman_gp4_support/meshes/gp4/visual/link_3_u.dae"/>
         </geometry>
-        <xacro:material_yaskawa_white/>
+        <xacro:material_yaskawa_blue/>
       </visual>
       <collision>
         <geometry>
-          <mesh filename="package://motoman_gp4_support/meshes/gp4/collision/link_3_u.dae"/>
+          <mesh filename="package://motoman_gp4_support/meshes/gp4/collision/link_3_u.stl"/>
         </geometry>
       </collision>
@@ -61,9 +61,9 @@
           <mesh filename="package://motoman_gp4_support/meshes/gp4/visual/link_4_r.dae"/>
         </geometry>
-        <xacro:material_yaskawa_white/>
+        <xacro:material_yaskawa_blue/>
       </visual>
       <collision>
         <geometry>
-          <mesh filename="package://motoman_gp4_support/meshes/gp4/collision/link_4_r.dae"/>
+          <mesh filename="package://motoman_gp4_support/meshes/gp4/collision/link_4_r.stl"/>
         </geometry>
       </collision>
@@ -74,9 +74,9 @@
           <mesh filename="package://motoman_gp4_support/meshes/gp4/visual/link_5_b.dae"/>
         </geometry>
-        <xacro:material_yaskawa_white/>
+        <xacro:material_yaskawa_blue/>
       </visual>
       <collision>
         <geometry>
-          <mesh filename="package://motoman_gp4_support/meshes/gp4/collision/link_5_b.dae"/>
+          <mesh filename="package://motoman_gp4_support/meshes/gp4/collision/link_5_b.stl"/>
         </geometry>
       </collision>
@@ -87,9 +87,9 @@
           <mesh filename="package://motoman_gp4_support/meshes/gp4/visual/link_6_t.dae"/>
         </geometry>
-        <xacro:material_yaskawa_white/>
+        <xacro:material_yaskawa_silver/>
       </visual>
       <collision>
         <geometry>
-          <mesh filename="package://motoman_gp4_support/meshes/gp4/collision/link_6_t.dae"/>
+          <mesh filename="package://motoman_gp4_support/meshes/gp4/collision/link_6_t.stl"/>
         </geometry>
       </collision>

Commit message: Update gp4_macro.xacro
Added the flange link between the joint_6_t and the tool0

File: motoman_gp4_support/urdf/gp4_macro.xacro (robot description, xacro)
@@ -95,5 +95,4 @@
       </collision>
     </link>
-    <link name="${prefix}tool0"/>
     <!-- end of link list -->
     <!-- joint list -->
@@ -140,10 +139,18 @@
       <limit lower="${radians(-455)}" upper="${radians(455)}" effort="16.46" velocity="${radians(1000)}"/>
     </joint>
-    <joint name="${prefix}joint_6_t-tool0" type="fixed">
+	<link name="${prefix}flange"/>
+    <joint name="${prefix}joint_6_t-flange" type="fixed">
       <origin xyz="0.072 0 0" rpy="${radians(180)} ${radians(-90)} 0"/>
       <parent link="${prefix}link_6_t"/>
+      <child link="${prefix}flange"/>
+    </joint>
+    <!-- end of joint list -->
+	<!-- default tool -->
+	<link name="${prefix}tool0"/>
+    <joint name="${prefix}flange-tool0" type="fixed">
+      <origin xyz="0 0 0" rpy="0 0 0"/>
+      <parent link="${prefix}flange"/>
       <child link="${prefix}tool0"/>
     </joint>
-    <!-- end of joint list -->
     <!-- ROS base_link to Robot Manufacturer World Coordinates transform -->
     <link name="${prefix}base" />

Commit message: Update gp4_macro.xacro
Corrected <tabs> for <spaces>

File: motoman_gp4_support/urdf/gp4_macro.xacro (robot description, xacro)
@@ -139,5 +139,5 @@
       <limit lower="${radians(-455)}" upper="${radians(455)}" effort="16.46" velocity="${radians(1000)}"/>
     </joint>
-	<link name="${prefix}flange"/>
+     <link name="${prefix}flange"/>
     <joint name="${prefix}joint_6_t-flange" type="fixed">
       <origin xyz="0.072 0 0" rpy="${radians(180)} ${radians(-90)} 0"/>
@@ -146,6 +146,6 @@
     </joint>
     <!-- end of joint list -->
-	<!-- default tool -->
-	<link name="${prefix}tool0"/>
+    <!-- default tool -->
+    <link name="${prefix}tool0"/>
     <joint name="${prefix}flange-tool0" type="fixed">
       <origin xyz="0 0 0" rpy="0 0 0"/>
