Commit message: fix velocity limits

File: motoman_gp8_support/urdf/gp8_macro.xacro (robot description, xacro)
@@ -110,5 +110,5 @@
         <origin xyz="0.040 0 0" rpy="0 0 0" />
         <axis xyz="0 1 0" />
-        <limit lower="-1.1344" upper="2.5307" effort="176.4" velocity="6.7495"/>
+        <limit lower="-1.1344" upper="2.5307" effort="176.4" velocity="6.7195"/>
     </joint>
     <joint name="${prefix}joint_3_u" type="revolute">
@@ -138,5 +138,5 @@
         <origin xyz="0 0 0" rpy="0 0 0" />
         <axis xyz="-1 0 0" />
-        <limit lower="-6.2944" upper="6.2944" effort="22.54" velocity="17.4845"/>
+        <limit lower="-6.2944" upper="6.2944" effort="22.54" velocity="17.4533"/>
     </joint>
     <joint name="${prefix}joint_6_t-tool0" type="fixed">

Commit message: urdf: include flange link, clean up whitespace

File: motoman_gp8_support/urdf/gp8_macro.xacro (robot description, xacro)
@@ -1,97 +1,97 @@
 <?xml version="1.0" ?>
 <robot xmlns:xacro="http://ros.org/wiki/xacro">
-<xacro:macro name="motoman_gp8" params="prefix">
+  <xacro:macro name="motoman_gp8" params="prefix">
     <xacro:include filename="$(find motoman_resources)/urdf/common_materials.xacro"/>
     <!-- link list -->
     <link name="${prefix}base_link">
-        <visual>
-            <geometry>
-                <mesh filename="package://motoman_gp8_support/meshes/visual/gp8_base_link.stl"/>
-            </geometry>
-            <xacro:material_yaskawa_blue/>
-        </visual>
-        <collision>
-            <geometry>
-                <mesh filename="package://motoman_gp8_support/meshes/collision/gp8_base_link.stl"/>
-            </geometry>
-        </collision>
+      <visual>
+        <geometry>
+          <mesh filename="package://motoman_gp8_support/meshes/visual/gp8_base_link.stl"/>
+        </geometry>
+        <xacro:material_yaskawa_blue/>
+      </visual>
+      <collision>
+        <geometry>
+          <mesh filename="package://motoman_gp8_support/meshes/collision/gp8_base_link.stl"/>
+        </geometry>
+      </collision>
     </link>
     <link name="${prefix}link_1_s">
-        <visual>
-            <geometry>
-                <mesh filename="package://motoman_gp8_support/meshes/visual/gp8_link_1_s.stl"/>
-            </geometry>
-            <xacro:material_yaskawa_blue/>
-        </visual>
-        <collision>
-            <geometry>
-                <mesh filename="package://motoman_gp8_support/meshes/collision/gp8_link_1_s.stl"/>
-            </geometry>
-        </collision>
+      <visual>
+        <geometry>
+          <mesh filename="package://motoman_gp8_support/meshes/visual/gp8_link_1_s.stl"/>
+        </geometry>
+        <xacro:material_yaskawa_blue/>
+      </visual>
+      <collision>
+        <geometry>
+          <mesh filename="package://motoman_gp8_support/meshes/collision/gp8_link_1_s.stl"/>
+        </geometry>
+      </collision>
     </link>
     <link name="${prefix}link_2_l">
-        <visual>
-            <geometry>
-                <mesh filename="package://motoman_gp8_support/meshes/visual/gp8_link_2_l.stl"/>
-            </geometry>
-            <xacro:material_yaskawa_blue/>
-        </visual>
-        <collision>
-            <geometry>
-                <mesh filename="package://motoman_gp8_support/meshes/collision/gp8_link_2_l.stl"/>
-            </geometry>
-        </collision>
+      <visual>
+        <geometry>
+          <mesh filename="package://motoman_gp8_support/meshes/visual/gp8_link_2_l.stl"/>
+        </geometry>
+        <xacro:material_yaskawa_blue/>
+      </visual>
+      <collision>
+        <geometry>
+          <mesh filename="package://motoman_gp8_support/meshes/collision/gp8_link_2_l.stl"/>
+        </geometry>
+      </collision>
     </link>
     <link name="${prefix}link_3_u">
-        <visual>
-            <geometry>
-                <mesh filename="package://motoman_gp8_support/meshes/visual/gp8_link_3_u.stl"/>
-            </geometry>
-            <xacro:material_yaskawa_blue/>
-        </visual>
-        <collision>
-            <geometry>
-                <mesh filename="package://motoman_gp8_support/meshes/collision/gp8_link_3_u.stl"/>
-            </geometry>
-        </collision>
+      <visual>
+        <geometry>
+          <mesh filename="package://motoman_gp8_support/meshes/visual/gp8_link_3_u.stl"/>
+        </geometry>
+        <xacro:material_yaskawa_blue/>
+      </visual>
+      <collision>
+        <geometry>
+          <mesh filename="package://motoman_gp8_support/meshes/collision/gp8_link_3_u.stl"/>
+        </geometry>
+      </collision>
     </link>
     <link name="${prefix}link_4_r">
-        <visual>
-            <geometry>
-                <mesh filename="package://motoman_gp8_support/meshes/visual/gp8_link_4_r.stl"/>
-            </geometry>
-            <xacro:material_yaskawa_blue/>
-        </visual>
-        <collision>
-            <geometry>
-                <mesh filename="package://motoman_gp8_support/meshes/collision/gp8_link_4_r.stl"/>
-            </geometry>
-        </collision>
+      <visual>
+        <geometry>
+          <mesh filename="package://motoman_gp8_support/meshes/visual/gp8_link_4_r.stl"/>
+        </geometry>
+        <xacro:material_yaskawa_blue/>
+      </visual>
+      <collision>
+        <geometry>
+          <mesh filename="package://motoman_gp8_support/meshes/collision/gp8_link_4_r.stl"/>
+        </geometry>
+      </collision>
     </link>
     <link name="${prefix}link_5_b">
-        <visual>
-            <geometry>
-                <mesh filename="package://motoman_gp8_support/meshes/visual/gp8_link_5_b.stl"/>
-            </geometry>
-            <xacro:material_yaskawa_blue/>
-        </visual>
-        <collision>
-            <geometry>
-                <mesh filename="package://motoman_gp8_support/meshes/collision/gp8_link_5_b.stl"/>
-            </geometry>
-        </collision>
+      <visual>
+        <geometry>
+          <mesh filename="package://motoman_gp8_support/meshes/visual/gp8_link_5_b.stl"/>
+        </geometry>
+        <xacro:material_yaskawa_blue/>
+      </visual>
+      <collision>
+        <geometry>
+          <mesh filename="package://motoman_gp8_support/meshes/collision/gp8_link_5_b.stl"/>
+        </geometry>
+      </collision>
     </link>
     <link name="${prefix}link_6_t">
-        <visual>
-            <geometry>
-                <mesh filename="package://motoman_gp8_support/meshes/visual/gp8_link_6_t.stl"/>
-            </geometry>
-            <xacro:material_yaskawa_blue/>
-        </visual>
-        <collision>
-            <geometry>
-                <mesh filename="package://motoman_gp8_support/meshes/collision/gp8_link_6_t.stl"/>
-            </geometry>
-        </collision>
+      <visual>
+        <geometry>
+          <mesh filename="package://motoman_gp8_support/meshes/visual/gp8_link_6_t.stl"/>
+        </geometry>
+        <xacro:material_yaskawa_blue/>
+      </visual>
+      <collision>
+        <geometry>
+          <mesh filename="package://motoman_gp8_support/meshes/collision/gp8_link_6_t.stl"/>
+        </geometry>
+      </collision>
     </link>
     <link name="${prefix}tool0"/>
@@ -99,58 +99,67 @@
     <!-- joint list -->
     <joint name="${prefix}joint_1_s" type="revolute">
-        <parent link="${prefix}base_link"/>
-        <child link="${prefix}link_1_s"/>
-        <origin xyz="0 0 0.330" rpy="0 0 0" />
-        <axis xyz="0 0 1" />
-        <limit lower="-2.9670" upper="2.9670" effort="150.92" velocity="7.9412"/>
+      <parent link="${prefix}base_link"/>
+      <child link="${prefix}link_1_s"/>
+      <origin xyz="0 0 0.330" rpy="0 0 0" />
+      <axis xyz="0 0 1" />
+      <limit lower="-2.9670" upper="2.9670" effort="150.92" velocity="7.9412"/>
     </joint>
     <joint name="${prefix}joint_2_l" type="revolute">
-        <parent link="${prefix}link_1_s"/>
-        <child link="${prefix}link_2_l"/>
-        <origin xyz="0.040 0 0" rpy="0 0 0" />
-        <axis xyz="0 1 0" />
-        <limit lower="-1.1344" upper="2.5307" effort="176.4" velocity="6.7195"/>
+      <parent link="${prefix}link_1_s"/>
+      <child link="${prefix}link_2_l"/>
+      <origin xyz="0.040 0 0" rpy="0 0 0" />
+      <axis xyz="0 1 0" />
+      <limit lower="-1.1344" upper="2.5307" effort="176.4" velocity="6.7195"/>
     </joint>
     <joint name="${prefix}joint_3_u" type="revolute">
-        <parent link="${prefix}link_2_l"/>
-        <child link="${prefix}link_3_u"/>
-        <origin xyz="0 0 0.345" rpy="0 0 0" />
-        <axis xyz="0 -1 0" />
-        <limit lower="-1.2217" upper="3.3161" effort="107.56" velocity="9.0757"/>
+      <parent link="${prefix}link_2_l"/>
+      <child link="${prefix}link_3_u"/>
+      <origin xyz="0 0 0.345" rpy="0 0 0" />
+      <axis xyz="0 -1 0" />
+      <limit lower="-1.2217" upper="3.3161" effort="107.56" velocity="9.0757"/>
     </joint>
     <joint name="${prefix}joint_4_r" type="revolute">
-        <parent link="${prefix}link_3_u"/>
-        <child link="${prefix}link_4_r"/>
-        <origin xyz="0.340 0 0.040" rpy="0 0 0" />
-        <axis xyz="-1 0 0" />
-        <limit lower="-3.3161" upper="3.3161" effort="55.86" velocity="9.5993"/>
+      <parent link="${prefix}link_3_u"/>
+      <child link="${prefix}link_4_r"/>
+      <origin xyz="0.340 0 0.040" rpy="0 0 0" />
+      <axis xyz="-1 0 0" />
+      <limit lower="-3.3161" upper="3.3161" effort="55.86" velocity="9.5993"/>
     </joint>
     <joint name="${prefix}joint_5_b" type="revolute">
-        <parent link="${prefix}link_4_r"/>
-        <child link="${prefix}link_5_b"/>
-        <origin xyz="0 0 0" rpy="0 0 0" />
-        <axis xyz="0 -1 0" />
-        <limit lower="-2.3561" upper="2.3561" effort="32.68" velocity="9.5993"/>
+      <parent link="${prefix}link_4_r"/>
+      <child link="${prefix}link_5_b"/>
+      <origin xyz="0 0 0" rpy="0 0 0" />
+      <axis xyz="0 -1 0" />
+      <limit lower="-2.3561" upper="2.3561" effort="32.68" velocity="9.5993"/>
     </joint>
     <joint name="${prefix}joint_6_t" type="revolute">
-        <parent link="${prefix}link_5_b"/>
-        <child link="${prefix}link_6_t"/>
-        <origin xyz="0 0 0" rpy="0 0 0" />
-        <axis xyz="-1 0 0" />
-        <limit lower="-6.2944" upper="6.2944" effort="22.54" velocity="17.4533"/>
-    </joint>
-    <joint name="${prefix}joint_6_t-tool0" type="fixed">
-        <origin xyz="0.080 0 0" rpy="3.1415926 -1.570796 0"/>
-        <parent link="${prefix}link_6_t"/>
-        <child link="${prefix}tool0"/>
+      <parent link="${prefix}link_5_b"/>
+      <child link="${prefix}link_6_t"/>
+      <origin xyz="0 0 0" rpy="0 0 0" />
+      <axis xyz="-1 0 0" />
+      <limit lower="-6.2944" upper="6.2944" effort="22.54" velocity="17.4533"/>
     </joint>
     <!-- end of joint list -->
+    <!-- ROS-Industrial 'flange' frame: attachment point for EEF models -->
+    <link name="${prefix}flange"/>
+    <joint name="${prefix}joint_6_t-flange" type="fixed">
+      <origin xyz="0.080 0 0" rpy="0 0 0"/>
+      <parent link="${prefix}link_6_t"/>
+      <child link="${prefix}flange"/>
+    </joint>
+    <!-- ROS-Industrial 'tool0' frame: all-zeros tool frame -->
+    <link name="${prefix}tool0"/>
+    <joint name="${prefix}flange-tool0" type="fixed">
+      <origin xyz="0 0 0" rpy="${radians(180)} ${radians(-90)} 0"/>
+      <parent link="${prefix}flange"/>
+      <child link="${prefix}tool0"/>
+    </joint>
     <!-- ROS base_link to Robot Manufacturer World Coordinates transform -->
     <link name="${prefix}base" />
     <joint name="${prefix}base_link-base" type="fixed">
-        <origin xyz="0 0 0.330" rpy="0 0 0"/>
-        <parent link="${prefix}base_link"/>
-        <child link="${prefix}base"/>
+      <origin xyz="0 0 0.330" rpy="0 0 0"/>
+      <parent link="${prefix}base_link"/>
+      <child link="${prefix}base"/>
     </joint>
-    </xacro:macro>
+  </xacro:macro>
 </robot>

Commit message: fix duplicate tool0 link

File: motoman_gp8_support/urdf/gp8_macro.xacro (robot description, xacro)
@@ -95,5 +95,4 @@
       </collision>
     </link>
-    <link name="${prefix}tool0"/>
     <!-- end of link list -->
     <!-- joint list -->

Commit message: fix small gp8 joint6 limit inaccuracy

File: motoman_gp8_support/urdf/gp8_macro.xacro (robot description, xacro)
@@ -137,5 +137,5 @@
       <origin xyz="0 0 0" rpy="0 0 0" />
       <axis xyz="-1 0 0" />
-      <limit lower="-6.2944" upper="6.2944" effort="22.54" velocity="17.4533"/>
+      <limit lower="-6.2831" upper="6.2831" effort="22.54" velocity="17.4533"/>
     </joint>
     <!-- end of joint list -->
