Commit message: fix some GP7 axis limit and velocity values based on datasheet

File: motoman_gp7_support/urdf/gp7_macro.xacro (robot description, xacro)
@@ -103,5 +103,5 @@
         <origin xyz="0 0 0.330" rpy="0 0 0" />
         <axis xyz="0 0 1" />
-        <limit lower="-2.9670" upper="2.9670" effort="212.66" velocity="6.5448"/>
+        <limit lower="-2.9670" upper="2.9670" effort="212.66" velocity="6.5449"/>
     </joint>
     <joint name="${prefix}joint_2_l" type="revolute">
@@ -138,5 +138,5 @@
         <origin xyz="0 0 0" rpy="0 0 0" />
         <axis xyz="-1 0 0" />
-        <limit lower="-6.2944" upper="6.2944" effort="22.54" velocity="17.4845"/>
+        <limit lower="-6.2831" upper="6.2831" effort="22.54" velocity="17.4533"/>
     </joint>
     <joint name="${prefix}joint_6_t-tool0" type="fixed">

Commit message: urdf: include flange link

File: motoman_gp7_support/urdf/gp7_macro.xacro (robot description, xacro)
@@ -1,5 +1,5 @@
 <?xml version="1.0" ?>
 <robot xmlns:xacro="http://ros.org/wiki/xacro">
-<xacro:macro name="motoman_gp7" params="prefix">
+    <xacro:macro name="motoman_gp7" params="prefix">
     <xacro:include filename="$(find motoman_resources)/urdf/common_materials.xacro"/>
     <!-- link list -->
@@ -95,5 +95,4 @@
         </collision>
     </link>
-    <link name="${prefix}tool0"/>
     <!-- end of link list -->
     <!-- joint list -->
@@ -140,10 +139,19 @@
         <limit lower="-6.2831" upper="6.2831" effort="22.54" velocity="17.4533"/>
     </joint>
-    <joint name="${prefix}joint_6_t-tool0" type="fixed">
-        <origin xyz="0.080 0 0" rpy="3.1415926 -1.570796 0"/>
+    <!-- end of joint list -->
+    <!-- ROS-Industrial 'flange' frame: attachment point for EEF models -->
+    <link name="${prefix}flange"/>
+    <joint name="${prefix}joint_6_t-flange" type="fixed">
+        <origin xyz="0.080 0 0" rpy="0 0 0"/>
         <parent link="${prefix}link_6_t"/>
+        <child link="${prefix}flange"/>
+    </joint>
+    <!-- ROS-Industrial 'tool0' frame: all-zeros tool frame -->
+    <link name="${prefix}tool0"/>
+    <joint name="${prefix}flange-tool0" type="fixed">
+        <origin xyz="0 0 0" rpy="${radians(180)} ${radians(-90)} 0"/>
+        <parent link="${prefix}flange"/>
         <child link="${prefix}tool0"/>
     </joint>
-    <!-- end of joint list -->
     <!-- ROS base_link to Robot Manufacturer World Coordinates transform -->
     <link name="${prefix}base" />
