Commit message: Correction of the model name to -b00
The DTP model was originally set as 'dtp-b10' but it should be 'dtp-b00'.  File names and references were corrected to 'dtp-b00'

File: motoman_hc10_support/urdf/hc10dtp_b00_macro.xacro (robot description, xacro)
@@ -1,5 +1,5 @@
 <?xml version="1.0" ?>
 <robot xmlns:xacro="http://ros.org/wiki/xacro">
-  <xacro:macro name="motoman_hc10dtp_b10" params="prefix">
+  <xacro:macro name="motoman_hc10dtp_b00" params="prefix">
     <xacro:include filename="$(find motoman_resources)/urdf/common_materials.xacro"/>
     <!-- link list -->
@@ -85,5 +85,5 @@
       <visual>
         <geometry>
-          <mesh filename="package://motoman_hc10_support/meshes/hc10dtp_b10/visual/link_6_t.dae"/>
+          <mesh filename="package://motoman_hc10_support/meshes/hc10dtp_b00/visual/link_6_t.dae"/>
         </geometry>
         <xacro:material_yaskawa_blue/>
@@ -91,5 +91,5 @@
       <collision>
         <geometry>
-          <mesh filename="package://motoman_hc10_support/meshes/hc10dtp_b10/collision/link_6_t.stl"/>
+          <mesh filename="package://motoman_hc10_support/meshes/hc10dtp_b00/collision/link_6_t.stl"/>
        </geometry>
       </collision>
