Commit message: rename base variant to HC20 DT; add DTP variant; add opw configs

File: motoman_hc20_support/urdf/hc20dtp_macro.xacro (robot description, xacro)
@@ -1,5 +1,5 @@
 <?xml version="1.0" ?>
 <robot xmlns:xacro="http://ros.org/wiki/xacro">
-  <xacro:macro name="motoman_hc20" params="prefix">
+  <xacro:macro name="motoman_hc20dtp" params="prefix">
     <xacro:include filename="$(find motoman_resources)/urdf/common_materials.xacro"/>
     <!-- link list -->
@@ -103,5 +103,5 @@
       <origin xyz="0 0 0.380" rpy="0 0 0" />
       <axis xyz="0 0 1" />
-      <limit lower="${radians(-180)}" upper="${radians(180)}" effort="917.28" velocity="${radians(80)}"/>
+      <limit lower="${radians(-210)}" upper="${radians(210)}" effort="917.28" velocity="${radians(80)}"/>
     </joint>
     <joint name="${prefix}joint_2_l" type="revolute">
